File: PCBs/rail/rail.kicad_pcb (KiCad board)
At the start: 2 copper layers, 58.5 x 34 mm, 7 parts

Commit message: Working UART input for basic control. All motors work. Next up: switch interrupts
Routing:
- net GND: vias 35 -> 39
Other:
- board text added: "TTK4900 RAIL MK1.2"
- board text removed: "TTK4900 RAIL MK1.1"
