File: PCBs/hand/IMU_assy.kicad_sch (KiCad schematic)
At the start: 5 parts, among them U5 LSM6DSMTR

Commit message: Updated ign with ever more variations of autosaves. Finished tracing hand, probably need new footprint for encoders. Next up: find footprints, redo IMU board
Parts:
- C21, C22: footprint Capacitor_SMD:C_0603_1608Metric -> Capacitor_SMD:C_0402_1005Metric
- R35: footprint Resistor_SMD:R_0805_2012Metric -> Resistor_SMD:R_0402_1005Metric
Changed lines of the file:
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@@
       (effects (font (size 1.27 1.27)))
     )
-    (property "Footprint" "Resistor_SMD:R_0805_2012Metric" (at 126.492 50.8 90)
+    (property "Footprint" "Resistor_SMD:R_0402_1005Metric" (at 126.492 50.8 90)
       (effects (font (size 1.27 1.27)) hide)
     )
@@
       (effects (font (size 1.27 1.27)) (justify left))
     )
-    (property "Footprint" "Capacitor_SMD:C_0603_1608Metric" (at 126.6952 82.55 0)
+    (property "Footprint" "Capacitor_SMD:C_0402_1005Metric" (at 126.6952 82.55 0)
       (effects (font (size 1.27 1.27)) hide)
     )
@@
       (effects (font (size 1.27 1.27)))
     )
-    (property "Footprint" "Resistor_SMD:R_0805_2012Metric" (at 123.952 50.8 90)
+    (property "Footprint" "Resistor_SMD:R_0402_1005Metric" (at 123.952 50.8 90)
       (effects (font (size 1.27 1.27)) hide)
     )
@@
       (effects (font (size 1.27 1.27)) (justify left))
     )
-    (property "Footprint" "Capacitor_SMD:C_0603_1608Metric" (at 83.5152 77.47 0)
-      (effects (font (size 1.27 1.27)) hide)
-    )
+    (property "Footprint" "Capacitor_SMD:C_0402_1005Metric" (at 83.5152 77.47 0)
+      (effects (font (size 1.27 1.27)) hide)
+    )

Commit message: Added pcb pdfs
Parts:
- renumbered R35 to R27, R35 to R31
Changed lines of the file:
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@@
   (symbol (lib_id "Device:R") (at 128.27 50.8 0) (unit 1)
     (in_bom yes) (on_board yes) (dnp no)
-    (property "Reference" "R35" (at 133.35 50.8 90)
+    (property "Reference" "R31" (at 133.35 50.8 90)
       (effects (font (size 1.27 1.27)))
     )
@@
     (instances
       (project "hand"
-        (path "/5df167e9-440d-40dc-8690-43ffe4e4c50d"
+        (path "/5df167e9-440d-40dc-8690-43ffe4e4c50d/75c4e4b3-beb7-4244-8d6d-015c4334d3f8"
+          (reference "R31") (unit 1)
+        )
+      )
+      (project "aux_hand_panel"
+        (path "/ef51f959-ef93-4df0-86d9-128ef67286ca/99710a32-e98a-46be-85cb-eaeb7f4354d6/75c4e4b3-beb7-4244-8d6d-015c4334d3f8"
           (reference "R35") (unit 1)
         )
-        (path "/5df167e9-440d-40dc-8690-43ffe4e4c50d/75c4e4b3-beb7-4244-8d6d-015c4334d3f8"
-          (reference "R31") (unit 1)
-        )
-      )
-      (project "aux_hand_panel"
-        (path "/ef51f959-ef93-4df0-86d9-128ef67286ca/99710a32-e98a-46be-85cb-eaeb7f4354d6/75c4e4b3-beb7-4244-8d6d-015c4334d3f8"
-          (reference "R35") (unit 1)
-        )
       )
     )
@@
   (symbol (lib_id "power:+3V3") (at 92.71 62.23 90) (unit 1)
     (in_bom yes) (on_board yes) (dnp no) (fields_autoplaced)
-    (property "Reference" "#PWR053" (at 96.52 62.23 0)
+    (property "Reference" "#PWR072" (at 96.52 62.23 0)
       (effects (font (size 1.27 1.27)) hide)
     )
@@
     (instances
       (project "hand"
-        (path "/5df167e9-440d-40dc-8690-43ffe4e4c50d"
-          (reference "#PWR053") (unit 1)
-        )
         (path "/5df167e9-440d-40dc-8690-43ffe4e4c50d/75c4e4b3-beb7-4244-8d6d-015c4334d3f8"
           (reference "#PWR072") (unit 1)
@@
   (symbol (lib_id "Device:R") (at 125.73 50.8 0) (unit 1)
     (in_bom yes) (on_board yes) (dnp no)
-    (property "Reference" "R35" (at 123.19 50.8 90)
+    (property "Reference" "R27" (at 123.19 50.8 90)
       (effects (font (size 1.27 1.27)))
     )
@@
     (instances
       (project "hand"
-        (path "/5df167e9-440d-40dc-8690-43ffe4e4c50d"
+        (path "/5df167e9-440d-40dc-8690-43ffe4e4c50d/75c4e4b3-beb7-4244-8d6d-015c4334d3f8"
+          (reference "R27") (unit 1)
+        )
+      )
+      (project "aux_hand_panel"
+        (path "/ef51f959-ef93-4df0-86d9-128ef67286ca/99710a32-e98a-46be-85cb-eaeb7f4354d6/75c4e4b3-beb7-4244-8d6d-015c4334d3f8"
           (reference "R35") (unit 1)
         )
-        (path "/5df167e9-440d-40dc-8690-43ffe4e4c50d/75c4e4b3-beb7-4244-8d6d-015c4334d3f8"
-          (reference "R27") (unit 1)
-        )
-      )
-      (project "aux_hand_panel"
-        (path "/ef51f959-ef93-4df0-86d9-128ef67286ca/99710a32-e98a-46be-85cb-eaeb7f4354d6/75c4e4b3-beb7-4244-8d6d-015c4334d3f8"
-          (reference "R35") (unit 1)
-        )
       )
     )
@@
   (symbol (lib_id "power:GND") (at 92.71 59.69 270) (unit 1)
     (in_bom yes) (on_board yes) (dnp no) (fields_autoplaced)
-    (property "Reference" "#PWR050" (at 86.36 59.69 0)
+    (property "Reference" "#PWR073" (at 86.36 59.69 0)
       (effects (font (size 1.27 1.27)) hide)
     )
@@
     (instances
       (project "hand"
-        (path "/5df167e9-440d-40dc-8690-43ffe4e4c50d"
-          (reference "#PWR050") (unit 1)
-        )
         (path "/5df167e9-440d-40dc-8690-43ffe4e4c50d/75c4e4b3-beb7-4244-8d6d-015c4334d3f8"
           (reference "#PWR073") (unit 1)
@@
   (symbol (lib_id "power:+3V3") (at 92.71 64.77 90) (unit 1)
     (in_bom yes) (on_board yes) (dnp no) (fields_autoplaced)
-    (property "Reference" "#PWR053" (at 96.52 64.77 0)
+    (property "Reference" "#PWR049" (at 96.52 64.77 0)
       (effects (font (size 1.27 1.27)) hide)
     )
@@
     (instances
       (project "hand"
-        (path "/5df167e9-440d-40dc-8690-43ffe4e4c50d"
-          (reference "#PWR053") (unit 1)
-        )
         (path "/5df167e9-440d-40dc-8690-43ffe4e4c50d/75c4e4b3-beb7-4244-8d6d-015c4334d3f8"
           (reference "#PWR049") (unit 1)
@@
     (instances
       (project "hand"
-        (path "/5df167e9-440d-40dc-8690-43ffe4e4c50d"
+        (path "/5df167e9-440d-40dc-8690-43ffe4e4c50d/75c4e4b3-beb7-4244-8d6d-015c4334d3f8"
           (reference "U5") (unit 1)
-        )
-        (path "/5df167e9-440d-40dc-8690-43ffe4e4c50d/75c4e4b3-beb7-4244-8d6d-015c4334d3f8"
-          (reference "U5") (unit 1)
