File: PCBs/hand/osc_rst_assy.kicad_sch (KiCad schematic)
At the start: 8 parts, among them J6 Conn_01x02

Commit message: Updated ign with ever more variations of autosaves. Finished tracing hand, probably need new footprint for encoders. Next up: find footprints, redo IMU board
Parts:
- BOOT0: footprint Connector_PinHeader_2.54mm:PinHeader_1x02_P2.54mm_Vertical -> Connector_PinHeader_2.54mm:PinHeader_1x02_P2.54mm_Horizontal
Changed lines of the file:
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@@
       (effects (font (size 1.27 1.27)))
     )
-    (property "Footprint" "Connector_PinHeader_2.54mm:PinHeader_1x02_P2.54mm_Vertical" (at 100.33 83.82 0)
+    (property "Footprint" "Connector_PinHeader_2.54mm:PinHeader_1x02_P2.54mm_Horizontal" (at 100.33 83.82 0)
       (effects (font (size 1.27 1.27)) hide)
     )

Commit message: Added pcb pdfs
Parts:
- renumbered BOOT0 to BOOT1, C2 to C19, R4 to R3
Changed lines of the file:
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@@
     (instances
       (project "hand"
-        (path "/5df167e9-440d-40dc-8690-43ffe4e4c50d"
-          (reference "XTAL1") (unit 1)
-        )
         (path "/5df167e9-440d-40dc-8690-43ffe4e4c50d/89b05129-cbc1-4cdc-a38b-34c728d41d99"
           (reference "XTAL1") (unit 1)
@@
   (symbol (lib_id "Device:C") (at 97.79 41.91 180) (unit 1)
     (in_bom yes) (on_board yes) (dnp no)
-    (property "Reference" "C2" (at 96.52 39.37 90)
+    (property "Reference" "C19" (at 96.52 39.37 90)
       (effects (font (size 1.27 1.27)))
     )
@@
     (instances
       (project "hand"
-        (path "/5df167e9-440d-40dc-8690-43ffe4e4c50d"
-          (reference "C2") (unit 1)
-        )
         (path "/5df167e9-440d-40dc-8690-43ffe4e4c50d/89b05129-cbc1-4cdc-a38b-34c728d41d99"
           (reference "C19") (unit 1)
@@
     (instances
       (project "hand"
-        (path "/5df167e9-440d-40dc-8690-43ffe4e4c50d"
+        (path "/5df167e9-440d-40dc-8690-43ffe4e4c50d/89b05129-cbc1-4cdc-a38b-34c728d41d99"
           (reference "C12") (unit 1)
         )
-        (path "/5df167e9-440d-40dc-8690-43ffe4e4c50d/89b05129-cbc1-4cdc-a38b-34c728d41d99"
-          (reference "C12") (unit 1)
-        )
       )
       (project "shoulder"
@@
     (instances
       (project "hand"
-        (path "/5df167e9-440d-40dc-8690-43ffe4e4c50d"
+        (path "/5df167e9-440d-40dc-8690-43ffe4e4c50d/89b05129-cbc1-4cdc-a38b-34c728d41d99"
           (reference "C11") (unit 1)
         )
-        (path "/5df167e9-440d-40dc-8690-43ffe4e4c50d/89b05129-cbc1-4cdc-a38b-34c728d41d99"
-          (reference "C11") (unit 1)
-        )
       )
       (project "shoulder"
@@
   (symbol (lib_id "Device:R") (at 102.87 60.96 270) (unit 1)
     (in_bom yes) (on_board yes) (dnp no)
-    (property "Reference" "R4" (at 104.14 55.88 0)
+    (property "Reference" "R3" (at 104.14 55.88 0)
       (effects (font (size 1.27 1.27)) (justify left))
     )
@@
     (instances
       (project "hand"
-        (path "/5df167e9-440d-40dc-8690-43ffe4e4c50d"
-          (reference "R4") (unit 1)
-        )
         (path "/5df167e9-440d-40dc-8690-43ffe4e4c50d/89b05129-cbc1-4cdc-a38b-34c728d41d99"
           (reference "R3") (unit 1)
@@
     (instances
       (project "hand"
-        (path "/5df167e9-440d-40dc-8690-43ffe4e4c50d"
-          (reference "R1") (unit 1)
-        )
         (path "/5df167e9-440d-40dc-8690-43ffe4e4c50d/89b05129-cbc1-4cdc-a38b-34c728d41d99"
           (reference "R1") (unit 1)
@@
   (symbol (lib_id "Jumper:Jumper_2_Open") (at 100.33 83.82 0) (unit 1)
     (in_bom yes) (on_board yes) (dnp no) (fields_autoplaced)
-    (property "Reference" "BOOT0" (at 100.33 77.47 0)
+    (property "Reference" "BOOT1" (at 100.33 77.47 0)
       (effects (font (size 1.27 1.27)))
     )
@@
     (instances
       (project "hand"
-        (path "/5df167e9-440d-40dc-8690-43ffe4e4c50d"
-          (reference "BOOT0") (unit 1)
-        )
         (path "/5df167e9-440d-40dc-8690-43ffe4e4c50d/89b05129-cbc1-4cdc-a38b-34c728d41d99"
           (reference "BOOT1") (unit 1)
