File: PCBs/hand/hand.kicad_sch (KiCad schematic)
At the start: 26 parts, among them U2 STM32F303RETx

Commit message: Updated ign with ever more variations of autosaves. Finished tracing hand, probably need new footprint for encoders. Next up: find footprints, redo IMU board
Parts:
- IMU_OPT1: footprint Connector_PinHeader_2.54mm:PinHeader_1x02_P2.54mm_Horizontal -> Connector_PinHeader_2.54mm:PinHeader_1x02_P2.54mm_Vertical
- PWR_CAN_IMU1: footprint Connector_PinHeader_2.54mm:PinHeader_2x04_P2.54mm_Horizontal -> Connector_PinHeader_2.54mm:PinHeader_2x04_P2.54mm_Vertical
- renumbered ENC2 to ENC1, ENC1 to ENC2
Connections:
- net +3V3: now also C4.1, C5.1
- net +48V: now also PWR_CAN_IMU1.2 (Pin_2); no longer PWR_CAN_IMU1.8 (Pin_8)
- net +5V: now also PWR_CAN_IMU1.1 (Pin_1); no longer PWR_CAN_IMU1.7 (Pin_7)
- net CANH: now also PWR_CAN_IMU1.6 (Pin_6); no longer PWR_CAN_IMU1.4 (Pin_4)
- net CANL: now also PWR_CAN_IMU1.4 (Pin_4); no longer PWR_CAN_IMU1.6 (Pin_6)
- net ENC1A: now also ENC1.5 (Pin_5); no longer ENC2.5 (Pin_5)
- net ENC1B: now also ENC1.3 (Pin_3); no longer ENC2.3 (Pin_3)
- net ENC2A: now also ENC2.5 (Pin_5); no longer ENC1.5 (Pin_5)
- net ENC2B: now also ENC2.3 (Pin_3); no longer ENC1.3 (Pin_3)
- net GND: now also PWR_CAN_IMU1.7 (Pin_7), PWR_CAN_IMU1.8 (Pin_8); no longer PWR_CAN_IMU1.1 (Pin_1), PWR_CAN_IMU1.2 (Pin_2)
- net I2C1_SCL: now also PWR_CAN_IMU1.3 (Pin_3)
- net I2C1_SDA: now also PWR_CAN_IMU1.5 (Pin_5)
- net I2C3_SCL: no longer PWR_CAN_IMU1.3 (Pin_3)
- net I2C3_SDA: no longer PWR_CAN_IMU1.5 (Pin_5)
- net IMU_INT3: now also IMU_OPT1.1 (Pin_1); no longer IMU_OPT1.2 (Pin_2)
- net OPT_SW2: now also IMU_OPT1.2 (Pin_2); no longer IMU_OPT1.1 (Pin_1)
- net at D1.2 (A), D2.2 (A): no longer C4.1, C5.1
Other:
- moved on the sheet: D1, D2, IMU_OPT1

Commit message: All revisions finished, MK1.1 ready for gerber generation
Parts:
- ENC1, ENC2: footprint Connector_PinHeader_2.54mm:PinHeader_1x05_P2.54mm_Vertical -> PINSOCKET:PinSocket_1x05_P2.54mm_Vertical
Changed lines of the file:
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@@
       (effects (font (size 1.27 1.27)))
     )
-    (property "Footprint" "Connector_PinHeader_2.54mm:PinHeader_1x05_P2.54mm_Vertical" (at 34.29 106.68 0)
+    (property "Footprint" "PINSOCKET:PinSocket_1x05_P2.54mm_Vertical" (at 34.29 106.68 0)
       (effects (font (size 1.27 1.27)) hide)
     )
@@
       (effects (font (size 1.27 1.27)))
     )
-    (property "Footprint" "Connector_PinHeader_2.54mm:PinHeader_1x05_P2.54mm_Vertical" (at 34.29 83.82 0)
-      (effects (font (size 1.27 1.27)) hide)
-    )
+    (property "Footprint" "PINSOCKET:PinSocket_1x05_P2.54mm_Vertical" (at 34.29 83.82 0)
+      (effects (font (size 1.27 1.27)) hide)
+    )

Commit message: Separated Hand B as separate Kicad project. Next up: gerber generation
Parts:
- removed H3, H4: MountingHole, MountingHole:MountingHole_2.7mm_M2.5, symbol Mechanical:MountingHole
Changed lines of the file:
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@@
-    )
-  )
-  (symbol (lib_id "Mechanical:MountingHole") (at 248.92 153.67 0) (unit 1)
-    (in_bom yes) (on_board yes) (dnp no) (fields_autoplaced)
-    (property "Reference" "H4" (at 251.46 152.4 0)
-      (effects (font (size 1.27 1.27)) (justify left))
-    )
-    (property "Value" "MountingHole" (at 251.46 154.94 0)
-      (effects (font (size 1.27 1.27)) (justify left))
-    )
-    (property "Footprint" "MountingHole:MountingHole_2.7mm_M2.5" (at 248.92 153.67 0)
-      (effects (font (size 1.27 1.27)) hide)
-    )
-    (property "Datasheet" "~" (at 248.92 153.67 0)
-      (effects (font (size 1.27 1.27)) hide)
-    )
-    (instances
-      (project "hand"
-        (path "/5df167e9-440d-40dc-8690-43ffe4e4c50d"
-          (reference "H4") (unit 1)
-        )
-      )
     )
   )
@@
         )
       )
-    )
-  )
-  (symbol (lib_id "Mechanical:MountingHole") (at 224.79 152.4 0) (unit 1)
-    (in_bom yes) (on_board yes) (dnp no) (fields_autoplaced)
-    (property "Reference" "H3" (at 227.33 151.13 0)
-      (effects (font (size 1.27 1.27)) (justify left))
-    )
-    (property "Value" "MountingHole" (at 227.33 153.67 0)
-      (effects (font (size 1.27 1.27)) (justify left))
-    )
-    (property "Footprint" "MountingHole:MountingHole_2.7mm_M2.5" (at 224.79 152.4 0)
-      (effects (font (size 1.27 1.27)) hide)
-    )
-    (property "Datasheet" "~" (at 224.79 152.4 0)
-      (effects (font (size 1.27 1.27)) hide)
-    )
-    (instances
-      (project "hand"
-        (path "/5df167e9-440d-40dc-8690-43ffe4e4c50d"
-          (reference "H3") (unit 1)
-        )
-      )

Commit message: merged changes from timertests, mostly documentation and such. Did not add tim6 config
Other:
- title: (none) -> Hand PCB
Changed lines of the file:
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@@
 (kicad_sch (version 20230121) (generator eeschema)
   (paper "A4")
+  (title_block
+    (title "Hand PCB")
+    (rev "Mk1.1")
+  )
   (junction (at 85.09 116.84) (diameter 0) (color 0 0 0 0)
   )
