File: PCBs/hand_B/hand_B.kicad_sch (KiCad schematic)
At the start: 5 parts

Commit message: Working UART input for basic control. All motors work. Next up: switch interrupts
Parts:
- R2: footprint Resistor_SMD:R_0402_1005Metric -> Resistor_SMD:R_0603_1608Metric
Changed lines of the file:
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@@
       (effects (font (size 1.27 1.27)) (justify left))
     )
-    (property "Footprint" "Resistor_SMD:R_0402_1005Metric" (at 125.222 80.01 90)
+    (property "Footprint" "Resistor_SMD:R_0603_1608Metric" (at 125.222 80.01 90)
       (effects (font (size 1.27 1.27)) hide)
     )

Commit message: Added pcb pdfs
Other:
- moved on the sheet: CON_B1, H3, H4, OPT1, R2
Changed lines of the file:
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@@
 (kicad_sch (version 20230121) (generator eeschema)
-  (paper "A4")
-  (wire (pts (xy 149.86 76.2) (xy 149.86 86.36))
+  (paper "A5")
+  (wire (pts (xy 114.3 57.15) (xy 114.3 67.31))
     (stroke (width 0) (type default))
   )
-  (wire (pts (xy 139.7 102.87) (xy 140.97 102.87))
+  (wire (pts (xy 104.14 83.82) (xy 105.41 83.82))
     (stroke (width 0) (type default))
   )
-  (wire (pts (xy 121.92 71.12) (xy 127 71.12))
+  (wire (pts (xy 86.36 52.07) (xy 91.44 52.07))
     (stroke (width 0) (type default))
   )
-  (wire (pts (xy 127 86.36) (xy 127 83.82))
+  (wire (pts (xy 91.44 67.31) (xy 91.44 64.77))
     (stroke (width 0) (type default))
   )
-  (wire (pts (xy 147.32 71.12) (xy 153.67 71.12))
+  (wire (pts (xy 111.76 52.07) (xy 118.11 52.07))
     (stroke (width 0) (type default))
   )
-  (wire (pts (xy 147.32 76.2) (xy 149.86 76.2))
+  (wire (pts (xy 111.76 57.15) (xy 114.3 57.15))
     (stroke (width 0) (type default))
   )
-  (wire (pts (xy 139.7 107.95) (xy 140.97 107.95))
+  (wire (pts (xy 104.14 88.9) (xy 105.41 88.9))
     (stroke (width 0) (type default))
   )
-  (wire (pts (xy 139.7 105.41) (xy 140.97 105.41))
+  (wire (pts (xy 104.14 86.36) (xy 105.41 86.36))
     (stroke (width 0) (type default))
   )
-  (wire (pts (xy 147.32 73.66) (xy 153.67 73.66))
+  (wire (pts (xy 111.76 54.61) (xy 118.11 54.61))
     (stroke (width 0) (type default))
   )
-  (label "0v" (at 140.97 107.95 0) (fields_autoplaced)
+  (label "0v" (at 105.41 88.9 0) (fields_autoplaced)
     (effects (font (size 1.27 1.27)) (justify left bottom))
   )
-  (label "OPT_B" (at 140.97 105.41 0) (fields_autoplaced)
+  (label "OPT_B" (at 105.41 86.36 0) (fields_autoplaced)
     (effects (font (size 1.27 1.27)) (justify left bottom))
   )
-  (label "0v" (at 127 86.36 270) (fields_autoplaced)
+  (label "0v" (at 91.44 67.31 270) (fields_autoplaced)
     (effects (font (size 1.27 1.27)) (justify right bottom))
   )
-  (label "5V" (at 121.92 71.12 0) (fields_autoplaced)
+  (label "5V" (at 86.36 52.07 0) (fields_autoplaced)
     (effects (font (size 1.27 1.27)) (justify left bottom))
   )
-  (label "5V" (at 140.97 102.87 0) (fields_autoplaced)
+  (label "5V" (at 105.41 83.82 0) (fields_autoplaced)
     (effects (font (size 1.27 1.27)) (justify left bottom))
   )
-  (label "5V" (at 153.67 71.12 0) (fields_autoplaced)
+  (label "5V" (at 118.11 52.07 0) (fields_autoplaced)
     (effects (font (size 1.27 1.27)) (justify left bottom))
   )
-  (label "0v" (at 149.86 86.36 270) (fields_autoplaced)
+  (label "0v" (at 114.3 67.31 270) (fields_autoplaced)
     (effects (font (size 1.27 1.27)) (justify right bottom))
   )
-  (label "OPT_B" (at 153.67 73.66 0) (fields_autoplaced)
+  (label "OPT_B" (at 118.11 54.61 0) (fields_autoplaced)
     (effects (font (size 1.27 1.27)) (justify left bottom))
   )
-  (symbol (lib_id "Device:R") (at 127 80.01 0) (unit 1)
+  (symbol (lib_id "Device:R") (at 91.44 60.96 0) (unit 1)
     (in_bom yes) (on_board yes) (dnp no)
-    (property "Reference" "R2" (at 125.73 85.09 90)
+    (property "Reference" "R2" (at 90.17 66.04 90)
       (effects (font (size 1.27 1.27)) (justify left))
     )
-    (property "Value" "220" (at 128.27 85.09 90)
+    (property "Value" "220" (at 92.71 66.04 90)
       (effects (font (size 1.27 1.27)) (justify left))
     )
-    (property "Footprint" "Resistor_SMD:R_0603_1608Metric" (at 125.222 80.01 90)
+    (property "Footprint" "Resistor_SMD:R_0603_1608Metric" (at 89.662 60.96 90)
       (effects (font (size 1.27 1.27)) hide)
     )
-    (property "Datasheet" "~" (at 127 80.01 0)
+    (property "Datasheet" "~" (at 91.44 60.96 0)
       (effects (font (size 1.27 1.27)) hide)
     )
@@
     )
   )
-  (symbol (lib_id "OPB971N51:OPB971N51") (at 137.16 73.66 0) (unit 1)
+  (symbol (lib_id "OPB971N51:OPB971N51") (at 101.6 54.61 0) (unit 1)
     (in_bom yes) (on_board yes) (dnp no) (fields_autoplaced)
-    (property "Reference" "OPT1" (at 137.16 66.04 0)
+    (property "Reference" "OPT1" (at 101.6 46.99 0)
       (effects (font (size 1.27 1.27)))
     )
-    (property "Value" "~" (at 135.89 80.01 0)
+    (property "Value" "~" (at 100.33 60.96 0)
       (effects (font (size 1.27 1.27)))
     )
-    (property "Footprint" "OPB971N51:OPB971N51" (at 135.89 80.01 0)
+    (property "Footprint" "OPB971N51:OPB971N51" (at 100.33 60.96 0)
       (effects (font (size 1.27 1.27)) hide)
     )
-    (property "Datasheet" "" (at 135.89 80.01 0)
+    (property "Datasheet" "" (at 100.33 60.96 0)
       (effects (font (size 1.27 1.27)) hide)
     )
@@
     )
   )
-  (symbol (lib_id "Mechanical:MountingHole") (at 209.55 137.16 0) (unit 1)
+  (symbol (lib_id "Mechanical:MountingHole") (at 149.86 97.79 0) (unit 1)
     (in_bom yes) (on_board yes) (dnp no) (fields_autoplaced)
-    (property "Reference" "H3" (at 212.09 135.89 0)
+    (property "Reference" "H3" (at 152.4 96.52 0)
       (effects (font (size 1.27 1.27)) (justify left))
     )
-    (property "Value" "MountingHole" (at 212.09 138.43 0)
+    (property "Value" "MountingHole" (at 152.4 99.06 0)
       (effects (font (size 1.27 1.27)) (justify left))
     )
-    (property "Footprint" "MountingHole:MountingHole_2.7mm_M2.5" (at 209.55 137.16 0)
+    (property "Footprint" "MountingHole:MountingHole_2.7mm_M2.5" (at 149.86 97.79 0)
       (effects (font (size 1.27 1.27)) hide)
     )
-    (property "Datasheet" "~" (at 209.55 137.16 0)
+    (property "Datasheet" "~" (at 149.86 97.79 0)
       (effects (font (size 1.27 1.27)) hide)
     )
@@
     )
   )
-  (symbol (lib_id "Mechanical:MountingHole") (at 233.68 138.43 0) (unit 1)
+  (symbol (lib_id "Mechanical:MountingHole") (at 173.99 99.06 0) (unit 1)
     (in_bom yes) (on_board yes) (dnp no) (fields_autoplaced)
-    (property "Reference" "H4" (at 236.22 137.16 0)
+    (property "Reference" "H4" (at 176.53 97.79 0)
       (effects (font (size 1.27 1.27)) (justify left))
     )
-    (property "Value" "MountingHole" (at 236.22 139.7 0)
+    (property "Value" "MountingHole" (at 176.53 100.33 0)
       (effects (font (size 1.27 1.27)) (justify left))
     )
-    (property "Footprint" "MountingHole:MountingHole_2.7mm_M2.5" (at 233.68 138.43 0)
+    (property "Footprint" "MountingHole:MountingHole_2.7mm_M2.5" (at 173.99 99.06 0)
       (effects (font (size 1.27 1.27)) hide)
     )
-    (property "Datasheet" "~" (at 233.68 138.43 0)
+    (property "Datasheet" "~" (at 173.99 99.06 0)
       (effects (font (size 1.27 1.27)) hide)
     )
@@
     )
   )
-  (symbol (lib_id "Connector_Generic:Conn_01x03") (at 134.62 105.41 180) (unit 1)
+  (symbol (lib_id "Connector_Generic:Conn_01x03") (at 99.06 86.36 180) (unit 1)
     (in_bom yes) (on_board yes) (dnp no) (fields_autoplaced)
-    (property "Reference" "CON_B1" (at 134.62 96.52 0)
+    (property "Reference" "CON_B1" (at 99.06 77.47 0)
       (effects (font (size 1.27 1.27)))
     )
-    (property "Value" "Conn_01x03" (at 134.62 99.06 0)
+    (property "Value" "Conn_01x03" (at 99.06 80.01 0)
       (effects (font (size 1.27 1.27)))
     )
-    (property "Footprint" "Connector_PinHeader_2.54mm:PinHeader_1x03_P2.54mm_Vertical" (at 134.62 105.41 0)
+    (property "Footprint" "Connector_PinHeader_2.54mm:PinHeader_1x03_P2.54mm_Vertical" (at 99.06 86.36 0)
       (effects (font (size 1.27 1.27)) hide)
     )
-    (property "Datasheet" "~" (at 134.62 105.41 0)
+    (property "Datasheet" "~" (at 99.06 86.36 0)
       (effects (font (size 1.27 1.27)) hide)
     )

Commit message: merged changes from timertests, mostly documentation and such. Did not add tim6 config
Other:
- title: (none) -> Hand B (opt sens) PCB
Changed lines of the file:
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@@
 (kicad_sch (version 20230121) (generator eeschema)
   (paper "A5")
+  (title_block
+    (title "Hand B (opt sens) PCB")
+    (rev "Mk1.1")
+  )
   (wire (pts (xy 114.3 57.15) (xy 114.3 67.31))
     (stroke (width 0) (type default))
