File: PCBs/imu/imu.kicad_sch (KiCad schematic)
At the start: 19 parts, among them U1 LSM6DSMTR, U2 ZMR330FTA

Commit message: merged changes from timertests, mostly documentation and such. Did not add tim6 config
Other:
- title: (none) -> IMU board PCB
Changed lines of the file:
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@@
 (kicad_sch (version 20230121) (generator eeschema)
   (paper "A5")
+  (title_block
+    (title "IMU board PCB")
+    (rev "Mk1.1")
+  )
   (junction (at 134.62 77.47) (diameter 0) (color 0 0 0 0)
   )
