File: PCBs/shoulder/can_assy.kicad_sch (KiCad schematic)
At the start: 4 parts, among them U1 TJA1057GT/3J

Commit message: merged changes from timertests, mostly documentation and such. Did not add tim6 config
Parts:
- renumbered C1 to C8, C3 to C9, U1 to U3
Changed lines of the file:
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@@
   (title_block
     (title "CAN assembly")
-    (rev "1.1")
+    (rev "Mk1.1")
   )
   (junction (at 74.93 69.85) (diameter 0) (color 0 0 0 0)
@@
   (symbol (lib_id "Device:C") (at 120.65 67.31 180) (unit 1)
     (in_bom yes) (on_board yes) (dnp no) (fields_autoplaced)
-    (property "Reference" "C3" (at 124.46 66.04 0)
+    (property "Reference" "C9" (at 124.46 66.04 0)
       (effects (font (size 1.27 1.27)) (justify right))
     )
@@
     (instances
       (project "shoulder"
-        (path "/5df167e9-440d-40dc-8690-43ffe4e4c50d"
-          (reference "C3") (unit 1)
-        )
-      )
-      (project "shoulder"
         (path "/dd0c7be8-ccf1-412d-960e-d6705c0e249b/38d303e4-1bac-45b0-bb1f-2ed94c6162e0"
           (reference "C9") (unit 1)
@@
   (symbol (lib_id "Device:C") (at 90.17 68.58 90) (unit 1)
     (in_bom yes) (on_board yes) (dnp no) (fields_autoplaced)
-    (property "Reference" "C1" (at 90.17 60.96 90)
+    (property "Reference" "C8" (at 90.17 60.96 90)
       (effects (font (size 1.27 1.27)))
     )
@@
     (instances
       (project "shoulder"
-        (path "/5df167e9-440d-40dc-8690-43ffe4e4c50d"
-          (reference "C1") (unit 1)
-        )
-      )
-      (project "shoulder"
         (path "/dd0c7be8-ccf1-412d-960e-d6705c0e249b/38d303e4-1bac-45b0-bb1f-2ed94c6162e0"
           (reference "C8") (unit 1)
@@
   (symbol (lib_id "TJA1057BT:TJA1057GT_3J") (at 106.68 76.2 180) (unit 1)
     (in_bom yes) (on_board yes) (dnp no) (fields_autoplaced)
-    (property "Reference" "U1" (at 106.68 62.23 0)
+    (property "Reference" "U3" (at 106.68 62.23 0)
       (effects (font (size 1.524 1.524)))
     )
@@
     (pin "8")
     (instances
-      (project "shoulder"
-        (path "/5df167e9-440d-40dc-8690-43ffe4e4c50d"
-          (reference "U1") (unit 1)
-        )
-      )
       (project "shoulder"
         (path "/dd0c7be8-ccf1-412d-960e-d6705c0e249b/38d303e4-1bac-45b0-bb1f-2ed94c6162e0"
@@
     (instances
       (project "shoulder"
-        (path "/5df167e9-440d-40dc-8690-43ffe4e4c50d"
-          (reference "CAN_TRM1") (unit 1)
-        )
-      )
-      (project "shoulder"
         (path "/dd0c7be8-ccf1-412d-960e-d6705c0e249b/38d303e4-1bac-45b0-bb1f-2ed94c6162e0"
