File: PCBs/shoulder/motor_assy.kicad_sch (KiCad schematic)
At the start: 14 parts, among them J1_MTR0 705430001, J2 Conn_01x07, J2_MTR1 705430001, Q1_RLY_CTRL Q_NIGBT_CGE

Commit message: merged changes from timertests, mostly documentation and such. Did not add tim6 config
Parts:
- renumbered C1_MTR0 to C_MTR1, C2_MTR1 to C_MTR2, J1_MTR0 to MTR1, J2_MTR1 to MTR2, Q1_RLY_CTRL to Q1_RLY_CTRL1, R1_IPROPI to R1_IPROPI1, R2_IPROPI to R2_IPROPI1
Changed lines of the file:
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@@
   (title_block
     (title "Motor driver assembly")
-    (rev "1.1")
+    (rev "Mk1.1")
   )
   (junction (at 107.95 110.49) (diameter 0) (color 0 0 0 0)
@@
   (symbol (lib_id "Device:R") (at 167.64 104.14 0) (unit 1)
     (in_bom yes) (on_board yes) (dnp no) (fields_autoplaced)
-    (property "Reference" "R1_IPROPI" (at 170.18 102.87 0)
+    (property "Reference" "R1_IPROPI1" (at 170.18 102.87 0)
       (effects (font (size 1.27 1.27)) (justify left))
     )
@@
     (instances
       (project "shoulder"
-        (path "/5df167e9-440d-40dc-8690-43ffe4e4c50d"
-          (reference "R1_IPROPI") (unit 1)
-        )
-        (path "/5df167e9-440d-40dc-8690-43ffe4e4c50d/710f463d-d939-4835-b806-0bed34cabba5"
-          (reference "R_IPROPI1") (unit 1)
-        )
-      )
-      (project "shoulder"
         (path "/dd0c7be8-ccf1-412d-960e-d6705c0e249b/23dd3c4a-da1f-44ef-acfb-616759cf75b9"
           (reference "R1_IPROPI1") (unit 1)
@@
   (symbol (lib_id "Device:C") (at 114.3 114.3 0) (unit 1)
     (in_bom yes) (on_board yes) (dnp no) (fields_autoplaced)
-    (property "Reference" "C2_MTR1" (at 118.11 113.03 0)
+    (property "Reference" "C_MTR2" (at 118.11 113.03 0)
       (effects (font (size 1.27 1.27)) (justify left))
     )
@@
     (instances
       (project "shoulder"
-        (path "/5df167e9-440d-40dc-8690-43ffe4e4c50d"
-          (reference "C2_MTR1") (unit 1)
-        )
-        (path "/5df167e9-440d-40dc-8690-43ffe4e4c50d/710f463d-d939-4835-b806-0bed34cabba5"
+        (path "/dd0c7be8-ccf1-412d-960e-d6705c0e249b/23dd3c4a-da1f-44ef-acfb-616759cf75b9"
           (reference "C_MTR2") (unit 1)
         )
       )
-      (project "shoulder"
-        (path "/dd0c7be8-ccf1-412d-960e-d6705c0e249b/23dd3c4a-da1f-44ef-acfb-616759cf75b9"
-          (reference "C_MTR2") (unit 1)
-        )
-      )
     )
   )
   (symbol (lib_id "Device:C") (at 114.3 85.09 0) (unit 1)
     (in_bom yes) (on_board yes) (dnp no) (fields_autoplaced)
-    (property "Reference" "C1_MTR0" (at 118.11 83.82 0)
+    (property "Reference" "C_MTR1" (at 118.11 83.82 0)
       (effects (font (size 1.27 1.27)) (justify left))
     )
@@
     (pin "2")
     (instances
-      (project "shoulder"
-        (path "/5df167e9-440d-40dc-8690-43ffe4e4c50d"
-          (reference "C1_MTR0") (unit 1)
-        )
-        (path "/5df167e9-440d-40dc-8690-43ffe4e4c50d/710f463d-d939-4835-b806-0bed34cabba5"
-          (reference "C_MTR1") (unit 1)
-        )
-      )
       (project "shoulder"
         (path "/dd0c7be8-ccf1-412d-960e-d6705c0e249b/23dd3c4a-da1f-44ef-acfb-616759cf75b9"
@@
     (instances
       (project "shoulder"
-        (path "/5df167e9-440d-40dc-8690-43ffe4e4c50d/710f463d-d939-4835-b806-0bed34cabba5"
-          (reference "MTR_DRV2") (unit 1)
-        )
-      )
-      (project "shoulder"
         (path "/dd0c7be8-ccf1-412d-960e-d6705c0e249b/23dd3c4a-da1f-44ef-acfb-616759cf75b9"
           (reference "MTR_DRV2") (unit 1)
@@
     (pin "4")
     (instances
-      (project "shoulder"
-        (path "/5df167e9-440d-40dc-8690-43ffe4e4c50d"
-          (reference "JV-3S-KT1") (unit 1)
-        )
-        (path "/5df167e9-440d-40dc-8690-43ffe4e4c50d/710f463d-d939-4835-b806-0bed34cabba5"
-          (reference "JV-3S-KT1") (unit 1)
-        )
-      )
       (project "shoulder"
         (path "/dd0c7be8-ccf1-412d-960e-d6705c0e249b/23dd3c4a-da1f-44ef-acfb-616759cf75b9"
@@
     (instances
       (project "shoulder"
-        (path "/5df167e9-440d-40dc-8690-43ffe4e4c50d/710f463d-d939-4835-b806-0bed34cabba5"
-          (reference "MTR_DRV1") (unit 1)
-        )
-      )
-      (project "shoulder"
         (path "/dd0c7be8-ccf1-412d-960e-d6705c0e249b/23dd3c4a-da1f-44ef-acfb-616759cf75b9"
           (reference "MTR_DRV1") (unit 1)
@@
     (instances
       (project "shoulder"
-        (path "/5df167e9-440d-40dc-8690-43ffe4e4c50d"
-          (reference "C4") (unit 1)
-        )
-        (path "/5df167e9-440d-40dc-8690-43ffe4e4c50d/710f463d-d939-4835-b806-0bed34cabba5"
-          (reference "C14") (unit 1)
-        )
-      )
-      (project "shoulder"
         (path "/dd0c7be8-ccf1-412d-960e-d6705c0e249b/23dd3c4a-da1f-44ef-acfb-616759cf75b9"
           (reference "C4") (unit 1)
@@
   (symbol (lib_id "Device:Q_NIGBT_CGE") (at 128.27 68.58 270) (mirror x) (unit 1)
     (in_bom yes) (on_board yes) (dnp no)
-    (property "Reference" "Q1_RLY_CTRL" (at 127 63.5 0)
+    (property "Reference" "Q1_RLY_CTRL1" (at 127 63.5 0)
       (effects (font (size 1.27 1.27)) (justify left))
     )
@@
     (instances
       (project "shoulder"
-        (path "/5df167e9-440d-40dc-8690-43ffe4e4c50d"
-          (reference "Q1_RLY_CTRL") (unit 1)
-        )
-        (path "/5df167e9-440d-40dc-8690-43ffe4e4c50d/710f463d-d939-4835-b806-0bed34cabba5"
-          (reference "RLY_CTRL1") (unit 1)
-        )
-      )
-      (project "shoulder"
         (path "/dd0c7be8-ccf1-412d-960e-d6705c0e249b/23dd3c4a-da1f-44ef-acfb-616759cf75b9"
           (reference "Q1_RLY_CTRL1") (unit 1)
@@
   (symbol (lib_id "70543-0001:705430001") (at 67.31 114.3 90) (unit 1)
     (in_bom yes) (on_board yes) (dnp no) (fields_autoplaced)
-    (property "Reference" "J2_MTR1" (at 73.66 113.03 90)
+    (property "Reference" "MTR2" (at 73.66 113.03 90)
       (effects (font (size 1.524 1.524)) (justify right))
     )
@@
     (instances
       (project "shoulder"
-        (path "/5df167e9-440d-40dc-8690-43ffe4e4c50d"
-          (reference "J2_MTR1") (unit 1)
-        )
-        (path "/5df167e9-440d-40dc-8690-43ffe4e4c50d/710f463d-d939-4835-b806-0bed34cabba5"
+        (path "/dd0c7be8-ccf1-412d-960e-d6705c0e249b/23dd3c4a-da1f-44ef-acfb-616759cf75b9"
           (reference "MTR2") (unit 1)
         )
       )
-      (project "shoulder"
-        (path "/dd0c7be8-ccf1-412d-960e-d6705c0e249b/23dd3c4a-da1f-44ef-acfb-616759cf75b9"
-          (reference "MTR2") (unit 1)
-        )
-      )
     )
   )
   (symbol (lib_name "705430001_1") (lib_id "70543-0001:705430001") (at 67.31 86.36 90) (unit 1)
     (in_bom yes) (on_board yes) (dnp no) (fields_autoplaced)
-    (property "Reference" "J1_MTR0" (at 73.66 85.09 90)
+    (property "Reference" "MTR1" (at 73.66 85.09 90)
       (effects (font (size 1.524 1.524)) (justify right))
     )
@@
     (instances
       (project "shoulder"
-        (path "/5df167e9-440d-40dc-8690-43ffe4e4c50d"
-          (reference "J1_MTR0") (unit 1)
-        )
-        (path "/5df167e9-440d-40dc-8690-43ffe4e4c50d/710f463d-d939-4835-b806-0bed34cabba5"
+        (path "/dd0c7be8-ccf1-412d-960e-d6705c0e249b/23dd3c4a-da1f-44ef-acfb-616759cf75b9"
           (reference "MTR1") (unit 1)
         )
       )
-      (project "shoulder"
-        (path "/dd0c7be8-ccf1-412d-960e-d6705c0e249b/23dd3c4a-da1f-44ef-acfb-616759cf75b9"
-          (reference "MTR1") (unit 1)
-        )
-      )
     )
   )
   (symbol (lib_id "Device:R") (at 167.64 132.08 0) (unit 1)
     (in_bom yes) (on_board yes) (dnp no) (fields_autoplaced)
-    (property "Reference" "R2_IPROPI" (at 170.18 130.81 0)
+    (property "Reference" "R2_IPROPI1" (at 170.18 130.81 0)
       (effects (font (size 1.27 1.27)) (justify left))
     )
@@
     (pin "2")
     (instances
-      (project "shoulder"
-        (path "/5df167e9-440d-40dc-8690-43ffe4e4c50d"
-          (reference "R2_IPROPI") (unit 1)
-        )
-        (path "/5df167e9-440d-40dc-8690-43ffe4e4c50d/710f463d-d939-4835-b806-0bed34cabba5"
-          (reference "R_IPROPI2") (unit 1)
-        )
-      )
       (project "shoulder"
         (path "/dd0c7be8-ccf1-412d-960e-d6705c0e249b/23dd3c4a-da1f-44ef-acfb-616759cf75b9"
@@
     (instances
       (project "shoulder"
-        (path "/5df167e9-440d-40dc-8690-43ffe4e4c50d"
-          (reference "C3") (unit 1)
-        )
-        (path "/5df167e9-440d-40dc-8690-43ffe4e4c50d/710f463d-d939-4835-b806-0bed34cabba5"
-          (reference "C13") (unit 1)
-        )
-      )
-      (project "shoulder"
         (path "/dd0c7be8-ccf1-412d-960e-d6705c0e249b/23dd3c4a-da1f-44ef-acfb-616759cf75b9"
           (reference "C3") (unit 1)
@@
     (instances
       (project "shoulder"
-        (path "/5df167e9-440d-40dc-8690-43ffe4e4c50d/710f463d-d939-4835-b806-0bed34cabba5"
-          (reference "RLY_CTL_DBG1") (unit 1)
-        )
-      )
-      (project "shoulder"
-        (path "/dd0c7be8-ccf1-412d-960e-d6705c0e249b/23dd3c4a-da1f-44ef-acfb-616759cf75b9"
+        (path "/dd0c7be8-ccf1-412d-960e-d6705c0e249b/23dd3c4a-da1f-44ef-acfb-616759cf75b9"
