File: PCBs/shoulder/osc_rst_assy.kicad_sch (KiCad schematic)
At the start: 8 parts, among them SW1 RESET

Commit message: merged changes from timertests, mostly documentation and such. Did not add tim6 config
Parts:
- renumbered BOOT0 to BOOT1, C2 to C5, C11 to C6, C12 to C7, R4 to R6, R1 to R7
Changed lines of the file:
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@@
   (title_block
     (title "Oscillator and reset assembly")
-    (rev "1.1")
+    (rev "Mk1.1")
   )
   (junction (at 99.06 50.8) (diameter 0) (color 0 0 0 0)
@@
   (symbol (lib_id "Device:C") (at 99.06 45.72 180) (unit 1)
     (in_bom yes) (on_board yes) (dnp no)
-    (property "Reference" "C2" (at 97.79 43.18 90)
+    (property "Reference" "C5" (at 97.79 43.18 90)
       (effects (font (size 1.27 1.27)))
     )
@@
     (pin "2")
     (instances
-      (project "shoulder"
-        (path "/5df167e9-440d-40dc-8690-43ffe4e4c50d"
-          (reference "C2") (unit 1)
-        )
-      )
       (project "shoulder"
         (path "/dd0c7be8-ccf1-412d-960e-d6705c0e249b/6be0f257-0828-42e7-90f4-699eb509c9fd"
@@
     (instances
       (project "shoulder"
-        (path "/5df167e9-440d-40dc-8690-43ffe4e4c50d"
-          (reference "SW1") (unit 1)
-        )
-      )
-      (project "shoulder"
         (path "/dd0c7be8-ccf1-412d-960e-d6705c0e249b/6be0f257-0828-42e7-90f4-699eb509c9fd"
           (reference "SW1") (unit 1)
@@
   (symbol (lib_id "Device:R") (at 104.14 64.77 270) (unit 1)
     (in_bom yes) (on_board yes) (dnp no)
-    (property "Reference" "R4" (at 105.41 59.69 0)
+    (property "Reference" "R6" (at 105.41 59.69 0)
       (effects (font (size 1.27 1.27)) (justify left))
     )
@@
     (instances
       (project "shoulder"
-        (path "/5df167e9-440d-40dc-8690-43ffe4e4c50d"
-          (reference "R4") (unit 1)
-        )
-      )
-      (project "shoulder"
         (path "/dd0c7be8-ccf1-412d-960e-d6705c0e249b/6be0f257-0828-42e7-90f4-699eb509c9fd"
           (reference "R6") (unit 1)
@@
   (symbol (lib_id "Device:R") (at 91.44 87.63 90) (unit 1)
     (in_bom yes) (on_board yes) (dnp no) (fields_autoplaced)
-    (property "Reference" "R1" (at 91.44 81.28 90)
+    (property "Reference" "R7" (at 91.44 81.28 90)
       (effects (font (size 1.27 1.27)))
     )
@@
     (pin "2")
     (instances
-      (project "shoulder"
-        (path "/5df167e9-440d-40dc-8690-43ffe4e4c50d"
-          (reference "R1") (unit 1)
-        )
-      )
       (project "shoulder"
         (path "/dd0c7be8-ccf1-412d-960e-d6705c0e249b/6be0f257-0828-42e7-90f4-699eb509c9fd"
@@
   (symbol (lib_id "Device:C") (at 93.98 64.77 270) (unit 1)
     (in_bom yes) (on_board yes) (dnp no)
-    (property "Reference" "C11" (at 91.44 66.04 90)
+    (property "Reference" "C6" (at 91.44 66.04 90)
       (effects (font (size 1.27 1.27)))
     )
@@
     (pin "2")
     (instances
-      (project "shoulder"
-        (path "/5df167e9-440d-40dc-8690-43ffe4e4c50d"
-          (reference "C11") (unit 1)
-        )
-      )
       (project "shoulder"
         (path "/dd0c7be8-ccf1-412d-960e-d6705c0e249b/6be0f257-0828-42e7-90f4-699eb509c9fd"
@@
     (instances
       (project "shoulder"
-        (path "/5df167e9-440d-40dc-8690-43ffe4e4c50d"
-          (reference "XTAL1") (unit 1)
-        )
-      )
-      (project "shoulder"
         (path "/dd0c7be8-ccf1-412d-960e-d6705c0e249b/6be0f257-0828-42e7-90f4-699eb509c9fd"
           (reference "XTAL1") (unit 1)
@@
   (symbol (lib_id "Device:C") (at 93.98 74.93 270) (unit 1)
     (in_bom yes) (on_board yes) (dnp no)
-    (property "Reference" "C12" (at 91.44 76.2 90)
+    (property "Reference" "C7" (at 91.44 76.2 90)
       (effects (font (size 1.27 1.27)))
     )
@@
     (pin "2")
     (instances
-      (project "shoulder"
-        (path "/5df167e9-440d-40dc-8690-43ffe4e4c50d"
-          (reference "C12") (unit 1)
-        )
-      )
       (project "shoulder"
         (path "/dd0c7be8-ccf1-412d-960e-d6705c0e249b/6be0f257-0828-42e7-90f4-699eb509c9fd"
@@
   (symbol (lib_id "Jumper:Jumper_2_Open") (at 101.6 87.63 0) (unit 1)
     (in_bom yes) (on_board yes) (dnp no) (fields_autoplaced)
-    (property "Reference" "BOOT0" (at 101.6 81.28 0)
+    (property "Reference" "BOOT1" (at 101.6 81.28 0)
       (effects (font (size 1.27 1.27)))
     )
@@
     (instances
       (project "shoulder"
-        (path "/5df167e9-440d-40dc-8690-43ffe4e4c50d"
-          (reference "BOOT0") (unit 1)
-        )
-      )
-      (project "shoulder"
-        (path "/dd0c7be8-ccf1-412d-960e-d6705c0e249b/6be0f257-0828-42e7-90f4-699eb509c9fd"
+        (path "/dd0c7be8-ccf1-412d-960e-d6705c0e249b/6be0f257-0828-42e7-90f4-699eb509c9fd"
