File: PCBs/torso/motor_assy.kicad_sch (KiCad schematic)
At the start: 14 parts, among them J1_MTR0 705430001, J2 Conn_01x07, J2_MTR1 705430001, Q1_RLY_CTRL Q_NIGBT_CGE

Commit message: Torso all but complete, making bogie before checking the last mark
Parts:
- removed C1_MTR0: 330muF, Capacitor_THT:CP_Radial_D16.0mm_P7.50mm, symbol Device:C
- removed C2_MTR1: 220muF, Capacitor_THT:CP_Radial_D10.0mm_P5.00mm, symbol Device:C
- removed J2_MTR1: 705430001, 70543-0001:70543-0001_MOL, symbol 70543-0001:705430001
- added C_MTR1, C_MTR2: 330uF, Capacitor_THT:CP_Radial_D16.0mm_P7.50mm, symbol Device:C_Polarized
- renumbered J1_MTR0 to MTR2, J2 to MTR_ASY_DBG1, Q1_RLY_CTRL to Q1_RLY_CTRL1, R1_IPROPI to R_IPROPI1, R2_IPROPI to R_IPROPI2
Connections:
- net Ground: now also C_MTR1.2, C_MTR2.2
- net at C3.2, C4.2, JV-3S-KT1.2 (COM)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: now also C_MTR1.1, C_MTR2.1
- net at MTR_DRV2.6 (OUT1): now also MTR2.2 (OUT)
- net at MTR_DRV2.8 (OUT2): now also MTR2.1 (IN)
- net MTR1_OUT: now reaches MTR_DRV1.6 (OUT1)
- net MTR1_OUT: no longer MTR2.2 (OUT)
- net MTR1_IN: now reaches MTR_DRV1.8 (OUT2)
- net MTR1_IN: no longer MTR2.1 (IN)
Other:
- title: Motor driver assembly -> (none)
- moved on the sheet: MTR2

Commit message: merged changes from timertests, mostly documentation and such. Did not add tim6 config
Other:
- title: (none) -> Motor assembly
Changed lines of the file:
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@@
 (kicad_sch (version 20230121) (generator eeschema)
   (paper "A4")
+  (title_block
+    (title "Motor assembly")
+    (rev "Mk1.2")
+  )
   (junction (at 107.95 110.49) (diameter 0) (color 0 0 0 0)
   )
