Commit message: various ROS improvements. Next up: PID tuning at varying voltages

File: code/ros/src/urdf/orca_description.urdf (robot description, URDF)
Before this commit: robot ttk4900_orca, 9 links, 8 joints
Links:
- link base_link: mass 15 -> None
Joints:
- joint joint_base_torso: limit lower=-1.65 upper=0 effort=70 velocity=0.1 -> lower=-1.40 upper=0 effort=100 velocity=0.1
- joint joint_hand_twist: limit lower=0.0 upper=0.0 effort=0.0 velocity=0.1 -> lower=0.0 upper=0.0 effort=100 velocity=3
- joint joint_lower_arm_hand: limit lower=-8 upper=2.5 effort=70 velocity=0.17 -> lower=-8 upper=2.5 effort=100 velocity=0.17
- joint joint_torso_upper_arm: limit lower=-1.2 upper=1.2 effort=70 velocity=0.17 -> lower=-1.3 upper=1.3 effort=100 velocity=0.17
- joint joint_twist_gripper0: limit lower=0.0 upper=0.04 effort=0.7 velocity=0.01 -> lower=0.0 upper=0.04 effort=100 velocity=0.01
- joint joint_twist_gripper1: limit lower=0.0 upper=0.04 effort=0.7 velocity=0.01 -> lower=0.0 upper=0.04 effort=100 velocity=0.01
- joint joint_upper_lower_arm: limit lower=-2.5 upper=2.5 effort=70 velocity=0.17 -> lower=-2.5 upper=2.5 effort=100 velocity=0.17

Commit message: pids are tuned, overall works better. Possibly reconsider elbow int action

File: code/ros/src/urdf/orca_description.urdf (robot description, URDF)
Before this commit: robot ttk4900_orca, 9 links, 8 joints
Joints:
- joint joint_torso_upper_arm: limit lower=-1.3 upper=1.3 effort=100 velocity=0.17 -> lower=-1.2 upper=1.2 effort=100 velocity=0.17

Commit message: minor code changes after testing at OV. IMPORTANT: IMU deactivated, shoulder limit to 1.5

File: code/ros/src/urdf/orca_description.urdf (robot description, URDF)
Before this commit: robot ttk4900_orca, 9 links, 8 joints
Joints:
- joint joint_hand_twist: limit lower=0.0 upper=0.0 effort=100 velocity=3 -> effort=100 velocity=3
- joint joint_torso_upper_arm: limit lower=-1.2 upper=1.2 effort=100 velocity=0.17 -> lower=-1.5 upper=1.5 effort=100 velocity=0.17

Commit message: got the pnp tutorial working with ORCA. Inconsistent IK solutions, and whether the cylinder loads or not is apparently random, but the code 'works'

File: code/ros/src/urdf/orca_description.urdf (robot description, URDF)
Before this commit: robot ttk4900_orca, 9 links, 8 joints
Links:
- link link_gripper0: geometry collision box size=0.038 0.013 0.15; visual box size=0.038 0.013 0.15
- link link_gripper1: geometry collision box size=0.038 0.013 0.15; visual box size=0.038 0.013 0.15
